File: hard/orangepi_ext/orangepi_ext.kicad_pcb (KiCad board)
At the start: 2 copper layers, 147 x 87 mm, 92 parts, among them J10 Power, J20 DEBUG, J21 EXT1, J22 EXT2, J40 DBG, J41 485-1, J42 232-1, J43 232-2, J50 YOUT, J51 VDD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

Commit message: orange pi extend hardware version 10 is outward processing
Parts:
- R52, R55: value 2.7k -> 10k
- turned U60 to 90 degrees
- turned U61 to 90 degrees
Routing:
- net GND: track 752.3 -> 734.2 mm, vias 10 -> 88
- net /DP2: track 35.7 -> 36.9 mm
- net VDD: vias 4 -> 5
- added copper zone on B.Cu, net GND
- added copper zone on F.Cu, net GND
